Commit message: Update mass and friction parameters

File: Software/Software/sbr_simulator/urdf/vehicle_urdf/urdf/vehicle_urdf.urdf (robot description, URDF)
Before this commit: robot vehicle_urdf, 3 links, 2 joints
Links:
- link base_link: mass 0.539786278718057 -> 1.5
- link left_link: mass 0.0181212751055899 -> 0.0145
- link right_wheel: mass 0.0181212751055898 -> 0.0145
